Commit message: ros2_control
urdf model -> gazebo simulation -> lidar simulation -> ros2 control simulation

!next up is hardware interface implementation

File: description/gazebo_control.xacro (robot description, xacro)
@@ -41,5 +41,5 @@
             <publish_distance>true</publish_distance>
             <odometry_frame>odom</odometry_frame>
-            <robot_base_frame>base_link</robot_base_frame>
+            <robot_base_frame>footprint_link</robot_base_frame>
         </plugin>
     </gazebo>

File: description/lidar.xacro (robot description, xacro)
@@ -4,5 +4,5 @@
         <parent link="chassis"/>
         <child link="lidar_frame"/>
-        <origin xyz="-0.2 0 0.3" rpy="0 0 0"/>
+        <origin xyz="-0.2 0 0.15" rpy="0 0 0"/>
     </joint>
     <link name="lidar_frame">

File: description/robot.urdf.xacro (robot description, xacro)
@@ -2,5 +2,10 @@
 <robot xmlns:xacro="http://www.ros.org/wiki/xacro"  name="robot">
     <xacro:include filename="robot_core.xacro" />
-    <xacro:include filename="gazebo_control.xacro" />
+    <xacro:if value="$(arg use_ros2_control)">
+        <xacro:include filename="ros2_control.xacro" />
+    </xacro:if>
+    <xacro:unless value="$(arg use_ros2_control)">
+        <xacro:include filename="gazebo_control.xacro" />
+    </xacro:unless>
     <xacro:include filename="lidar.xacro" />
 </robot>

File: description/robot_core.xacro (robot description, xacro)
@@ -20,5 +20,4 @@
     </joint> -->
     <link name="footprint_link">
-        <origin xyz="0 0 0" rpy="0 0 0" />
     </link>
     <!-- BASE LINK -->
@@ -34,9 +33,8 @@
         <parent link="base_link"/>
         <child link="chassis"/>
-        <origin xyz="0.3 0 0"/>
+        <origin xyz="0.3 0 0.125"/>
     </joint>
     <link name="chassis">
         <visual>
-            <origin xyz="0 0 0.125"/>
             <geometry>
                 <box size="1 0.2 0.25"/>
@@ -45,5 +43,4 @@
         </visual>
         <collision>
-            <origin xyz="0 0 0.125"/>
             <geometry>
                 <box size="1 0.2 0.25"/>
@@ -51,5 +48,5 @@
         </collision>
         <xacro:inertial_box mass="20" x="1" y="0.2" z="0.25">
-            <origin xyz="0 0 0.125" rpy="0 0 0"/>
+            <origin xyz="0 0 0" rpy="0 0 0"/>
         </xacro:inertial_box>
     </link>
@@ -61,8 +58,8 @@
     <!-- FRONT LEFT WHEEL -->
     <!-- steering -->
-    <joint name="left_steering_joint" type="revolute">
-        <parent link="chassis"/>
+    <joint name="front_left_steering_joint" type="revolute">
+        <parent link="base_link"/>
         <child link="left_steering_link"/>
-        <origin xyz="0.3 0.21 0" rpy="0 0 0"/>
+        <origin xyz="0.6 0.21 0" rpy="0 0 0"/>
         <axis xyz="0 0 1"/>
         <limit lower="-${pi/8}" upper="${pi/8}" effort="20" velocity="5"/> <!-- TODO -->
@@ -80,5 +77,5 @@
         <axis xyz="0 0 -1"/>
         <dynamics friction="0.8" damping="0.5" /> <!-- TODO -->
-        <limit lower="-3.14159" upper="3.14159" effort="0" velocity="-1" /> <!-- TODO -->
+        <limit lower="-3.14159" upper="3.14159" effort="0" velocity="1" /> <!-- TODO -->
     </joint>
     <link name="front_left_wheel">
@@ -107,8 +104,8 @@
     <!-- FRONT RIGHT WHEEL -->
     <!-- steering -->
-    <joint name="right_steering_joint" type="revolute">
-        <parent link="chassis"/>
+    <joint name="front_right_steering_joint" type="revolute">
+        <parent link="base_link"/>
         <child link="right_steering_link"/>
-        <origin xyz="0.3 -0.21 0" rpy="0 0 0"/>
+        <origin xyz="0.6 -0.21 0" rpy="0 0 0"/>
         <axis xyz="0 0 1"/>
         <limit lower="-${pi/8}" upper="${pi/8}" effort="20" velocity="5"/> <!-- TODO -->
@@ -126,5 +123,5 @@
         <axis xyz="0 0 1"/>
         <dynamics friction="0.8" damping="0.5" /> <!-- TODO -->
-        <limit lower="-3.14159" upper="3.14159" effort="0" velocity="-1" /> <!-- TODO -->
+        <limit lower="-3.14159" upper="3.14159" effort="0" velocity="1" /> <!-- TODO -->
     </joint>
     <link name="front_right_wheel">
@@ -154,10 +151,10 @@
     <!-- rotation -->
     <joint name="rear_left_wheel_joint" type="continuous">
-        <parent link="chassis"/>
+        <parent link="base_link"/>
         <child link="rear_left_wheel"/>
-        <origin xyz="-0.3 0.21 0" rpy="${pi/2} 0 0"/>
+        <origin xyz="0 0.21 0" rpy="${pi/2} 0 0"/>
         <axis xyz="0 0 -1"/>
         <dynamics friction="0.8" damping="0.5" /> <!-- TODO -->
-        <limit lower="-3.14159" upper="3.14159" effort="200" velocity="-1" /> <!-- TODO -->
+        <limit lower="-3.14159" upper="3.14159" effort="200" velocity="1" /> <!-- TODO -->
     </joint>
     <link name="rear_left_wheel">
@@ -181,16 +178,16 @@
     <gazebo reference="rear_left_wheel">
         <material>Gazebo/Black</material>
-        <mu1>2.5</mu1> <!-- TODO -->
-        <mu2>2.5</mu2> <!-- TODO -->
+        <mu1>10</mu1> <!-- TODO -->
+        <mu2>10</mu2> <!-- TODO -->
     </gazebo>
     <!-- REAR RIGHT WHEEL -->
     <!-- rotation -->
     <joint name="rear_right_wheel_joint" type="continuous">
-        <parent link="chassis"/>
+        <parent link="base_link"/>
         <child link="rear_right_wheel"/>
-        <origin xyz="-0.3 -0.21 0" rpy="-${pi/2} 0 0"/>
-        <axis xyz="0 0 1"/>
-        <dynamics friction="0.8" damping="0.5" /> <!-- TODO -->
-        <limit lower="-3.14159" upper="3.14159" effort="200" velocity="-1" /> <!-- TODO -->
+        <origin xyz="0 -0.21 0" rpy="-${pi/2} 0 0"/>
+        <axis xyz="0 0 1"/>
+        <dynamics friction="0.8" damping="0.5" /> <!-- TODO -->
+        <limit lower="-3.14159" upper="3.14159" effort="200" velocity="1" /> <!-- TODO -->
     </joint>
     <link name="rear_right_wheel">
@@ -214,6 +211,6 @@
     <gazebo reference="rear_right_wheel">
         <material>Gazebo/Black</material>
-        <mu1>2.5</mu1> <!-- TODO -->
-        <mu2>2.5</mu2> <!-- TODO -->
+        <mu1>10</mu1> <!-- TODO -->
+        <mu2>10</mu2> <!-- TODO -->
     </gazebo>
     <!-- VIRTUAL STEERING WHEEL -->
